File: 8330EVA-kicad/DAC.sch (KiCad schematic (older format))
At the start: 7 parts

Commit message: 修复若干ERC未连接错误
Parts:
- gave numbers to parts that had none: 7
Changed lines of the file:
@@
 $EndDescr
 $Comp
-L 8330_EVA-extra:AD5312 U?
+L 8330_EVA-extra:AD5312 U5
 U 1 1 5C0CBF97
 P 5700 3400
-F 0 "U?" H 5700 3915 50  0000 C CNN
+F 0 "U5" H 5700 3915 50  0000 C CNN
 F 1 "AD5312" H 5700 3824 50  0000 C CNN
 F 2 "" H 5700 2950 50  0001 C CNN
@@
 $EndComp
 $Comp
-L Reference_Voltage:REF192 U?
+L Reference_Voltage:REF192 U6
 U 1 1 5C0CD4C7
 P 6750 2700
-F 0 "U?" V 6654 2356 50  0000 R CNN
+F 0 "U6" V 6654 2356 50  0000 R CNN
 F 1 "REF192" V 6745 2356 50  0000 R CNN
 F 2 "" H 6750 2650 50  0001 C CIN
@@
 	6050 2700 6350 2700
 $Comp
-L Device:C C?
+L Device:C C40
 U 1 1 5C0D77AA
 P 7500 2700
-F 0 "C?" H 7615 2746 50  0000 L CNN
+F 0 "C40" H 7615 2746 50  0000 L CNN
 F 1 "10u" H 7615 2655 50  0000 L CNN
 F 2 "" H 7538 2550 50  0001 C CNN
@@
 Connection ~ 6750 2200
 $Comp
-L Device:C C?
+L Device:C C41
 U 1 1 5C0D8F63
 P 7950 2700
-F 0 "C?" H 8065 2746 50  0000 L CNN
+F 0 "C41" H 8065 2746 50  0000 L CNN
 F 1 "0.1u" H 8065 2655 50  0000 L CNN
 F 2 "" H 7988 2550 50  0001 C CNN
@@
 Connection ~ 7500 3000
 $Comp
-L Device:C C?
+L Device:C C38
 U 1 1 5C0D9F40
 P 6900 3200
-F 0 "C?" V 6648 3200 50  0000 C CNN
+F 0 "C38" V 6648 3200 50  0000 C CNN
 F 1 "1u" V 6739 3200 50  0000 C CNN
 F 2 "" H 6938 3050 50  0001 C CNN
@@
 	6750 3200 6750 3500
 $Comp
-L Device:C C?
+L Device:C C39
 U 1 1 5C0DA65E
 P 6900 3500
-F 0 "C?" V 6648 3500 50  0000 C CNN
+F 0 "C39" V 6648 3500 50  0000 C CNN
 F 1 "0.1u" V 6739 3500 50  0000 C CNN
 F 2 "" H 6938 3350 50  0001 C CNN
@@
 	7050 3500 7050 4250
 $Comp
-L Device:C C?
+L Device:C C37
 U 1 1 5C0DB093
 P 4650 3050
-F 0 "C?" H 4765 3096 50  0000 L CNN
+F 0 "C37" H 4765 3096 50  0000 L CNN
 F 1 "1u" H 4765 3005 50  0000 L CNN
 F 2 "" H 4688 2900 50  0001 C CNN

Commit message: 为变压器制作封装
Parts:
- C37, C38, C39, C40, C41: footprint (none) -> Capacitor_SMD:C_0603_1608Metric_Pad1.05x0.95mm_HandSolder
- U5: footprint (none) -> Package_SO:MSOP-10_3x3mm_P0.5mm
- U6: footprint (none) -> Package_SO:SOIC-8_3.9x4.9mm_P1.27mm
Changed lines of the file:
@@
 F 0 "U5" H 5700 3915 50  0000 C CNN
 F 1 "AD5312" H 5700 3824 50  0000 C CNN
-F 2 "" H 5700 2950 50  0001 C CNN
+F 2 "Package_SO:MSOP-10_3x3mm_P0.5mm" H 5700 2950 50  0001 C CNN
 F 3 "" H 5700 2950 50  0001 C CNN
 	1    5700 3400
@@
 F 0 "U6" V 6654 2356 50  0000 R CNN
 F 1 "REF192" V 6745 2356 50  0000 R CNN
-F 2 "" H 6750 2650 50  0001 C CIN
+F 2 "Package_SO:SOIC-8_3.9x4.9mm_P1.27mm" H 6750 2650 50  0001 C CIN
 F 3 "http://www.analog.com/static/imported-files/data_sheets/REF19xSeries.pdf" H 6750 2650 50  0001 C CIN
 	1    6750 2700
@@
 F 0 "C40" H 7615 2746 50  0000 L CNN
 F 1 "10u" H 7615 2655 50  0000 L CNN
-F 2 "" H 7538 2550 50  0001 C CNN
+F 2 "Capacitor_SMD:C_0603_1608Metric_Pad1.05x0.95mm_HandSolder" H 7538 2550 50  0001 C CNN
 F 3 "~" H 7500 2700 50  0001 C CNN
 	1    7500 2700
@@
 F 0 "C41" H 8065 2746 50  0000 L CNN
 F 1 "0.1u" H 8065 2655 50  0000 L CNN
-F 2 "" H 7988 2550 50  0001 C CNN
+F 2 "Capacitor_SMD:C_0603_1608Metric_Pad1.05x0.95mm_HandSolder" H 7988 2550 50  0001 C CNN
 F 3 "~" H 7950 2700 50  0001 C CNN
 	1    7950 2700
@@
 F 0 "C38" V 6648 3200 50  0000 C CNN
 F 1 "1u" V 6739 3200 50  0000 C CNN
-F 2 "" H 6938 3050 50  0001 C CNN
+F 2 "Capacitor_SMD:C_0603_1608Metric_Pad1.05x0.95mm_HandSolder" H 6938 3050 50  0001 C CNN
 F 3 "~" H 6900 3200 50  0001 C CNN
 	1    6900 3200
@@
 F 0 "C39" V 6648 3500 50  0000 C CNN
 F 1 "0.1u" V 6739 3500 50  0000 C CNN
-F 2 "" H 6938 3350 50  0001 C CNN
+F 2 "Capacitor_SMD:C_0603_1608Metric_Pad1.05x0.95mm_HandSolder" H 6938 3350 50  0001 C CNN
 F 3 "~" H 6900 3500 50  0001 C CNN
 	1    6900 3500
@@
 F 0 "C37" H 4765 3096 50  0000 L CNN
 F 1 "1u" H 4765 3005 50  0000 L CNN
-F 2 "" H 4688 2900 50  0001 C CNN
+F 2 "Capacitor_SMD:C_0603_1608Metric_Pad1.05x0.95mm_HandSolder" H 4688 2900 50  0001 C CNN
 F 3 "~" H 4650 3050 50  0001 C CNN
 	1    4650 3050
