File: 8330EVA-kicad/SingleToDifferential.sch (KiCad schematic (older format))
At the start: 10 parts

Commit message: 修复若干ERC未连接错误
Parts:
- gave numbers to parts that had none: 10
Changed lines of the file:
@@
 $EndDescr
 $Comp
-L 8330_EVA-extra:AD8131 U?
+L 8330_EVA-extra:AD8131 U4
 U 1 1 5BFB9A92
 P 5200 3450
-F 0 "U?" H 5175 3865 50  0000 C CNN
+F 0 "U4" H 5175 3865 50  0000 C CNN
 F 1 "AD8131" H 5175 3774 50  0000 C CNN
 F 2 "Package_SO:SOIC-8_3.9x4.9mm_P1.27mm" H 5350 3050 50  0001 C CNN
@@
 Ground
 $Comp
-L Device:R R?
+L Device:R R7
 U 1 1 5BFB9A9A
 P 3900 3650
-F 0 "R?" H 3750 3750 50  0000 L CNN
+F 0 "R7" H 3750 3750 50  0000 L CNN
 F 1 "49.9" H 3800 3600 50  0000 L CNN
 F 2 "" V 3830 3650 50  0001 C CNN
@@
 	3900 3300 3900 3500
 $Comp
-L power:Earth #PWR?
+L power:Earth #PWR0102
 U 1 1 5BFB9AA2
 P 3900 4000
-F 0 "#PWR?" H 3900 3750 50  0001 C CNN
+F 0 "#PWR0102" H 3900 3750 50  0001 C CNN
 F 1 "Earth" H 3900 3850 50  0001 C CNN
 F 2 "" H 3900 4000 50  0001 C CNN
@@
 Connection ~ 3900 3300
 $Comp
-L Device:C C?
+L Device:C C31
 U 1 1 5BFB9AAC
 P 4150 3650
-F 0 "C?" H 4250 3550 50  0000 R CNN
+F 0 "C31" H 4250 3550 50  0000 R CNN
 F 1 "0.1u" H 4200 3750 50  0000 R CNN
 F 2 "" H 4188 3500 50  0001 C CNN
@@
 	3900 3900 3900 4000
 $Comp
-L Device:R R?
+L Device:R R8
 U 1 1 5BFB9AB7
 P 4400 3650
-F 0 "R?" H 4250 3750 50  0000 L CNN
+F 0 "R8" H 4250 3750 50  0000 L CNN
 F 1 "24.9" H 4300 3600 50  0000 L CNN
 F 2 "" V 4330 3650 50  0001 C CNN
@@
 	4700 3500 4650 3500
 $Comp
-L Device:C C?
+L Device:C C34
 U 1 1 5BFB9AC0
 P 4900 4550
-F 0 "C?" H 5000 4450 50  0000 R CNN
+F 0 "C34" H 5000 4450 50  0000 R CNN
 F 1 "0.1u" H 4950 4650 50  0000 R CNN
 F 2 "" H 4938 4400 50  0001 C CNN
@@
 $EndComp
 $Comp
-L Device:C C?
+L Device:C C35
 U 1 1 5BFB9AC6
 P 5300 4550
-F 0 "C?" H 5400 4450 50  0000 R CNN
+F 0 "C35" H 5400 4450 50  0000 R CNN
 F 1 "10u" H 5350 4650 50  0000 R CNN
 F 2 "" H 5338 4400 50  0001 C CNN
@@
 	3400 3900 3900 3900
 $Comp
-L power:Earth #PWR?
+L power:Earth #PWR0103
 U 1 1 5BFB9AD5
 P 5100 5000
-F 0 "#PWR?" H 5100 4750 50  0001 C CNN
+F 0 "#PWR0103" H 5100 4750 50  0001 C CNN
 F 1 "Earth" H 5100 4850 50  0001 C CNN
 F 2 "" H 5100 5000 50  0001 C CNN
@@
 	5100 5000 5100 4850
 $Comp
-L Device:C C?
+L Device:C C36
 U 1 1 5BFB9AE1
 P 5950 3750
-F 0 "C?" H 6050 3650 50  0000 R CNN
+F 0 "C36" H 6050 3650 50  0000 R CNN
 F 1 "10n" H 6000 3850 50  0000 R CNN
 F 2 "" H 5988 3600 50  0001 C CNN
@@
 	5950 3500 6200 3500
 $Comp
-L power:Earth #PWR?
+L power:Earth #PWR0104
 U 1 1 5BFB9AEA
 P 5950 4050
-F 0 "#PWR?" H 5950 3800 50  0001 C CNN
+F 0 "#PWR0104" H 5950 3800 50  0001 C CNN
 F 1 "Earth" H 5950 3900 50  0001 C CNN
 F 2 "" H 5950 4050 50  0001 C CNN
@@
 	3900 2950 5650 2950
 $Comp
-L Device:C C?
+L Device:C C30
 U 1 1 5BFB9AF8
 P 4050 2700
-F 0 "C?" H 4150 2600 50  0000 R CNN
+F 0 "C30" H 4150 2600 50  0000 R CNN
 F 1 "0.1u" H 4100 2800 50  0000 R CNN
 F 2 "" H 4088 2550 50  0001 C CNN
@@
 $EndComp
 $Comp
-L Device:C C?
+L Device:C C32
 U 1 1 5BFB9AFE
 P 4300 2700
-F 0 "C?" H 4400 2600 50  0000 R CNN
+F 0 "C32" H 4400 2600 50  0000 R CNN
 F 1 "10u" H 4350 2800 50  0000 R CNN
 F 2 "" H 4338 2550 50  0001 C CNN
@@
 Connection ~ 4150 3900
 $Comp
-L Device:C C?
+L Device:C C33
 U 1 1 5BFB9B08
 P 4600 3650
-F 0 "C?" H 4700 3550 50  0000 R CNN
+F 0 "C33" H 4700 3550 50  0000 R CNN
 F 1 "10n" H 4650 3750 50  0000 R CNN
 F 2 "" H 4638 3500 50  0001 C CNN

Commit message: 为变压器制作封装
Parts:
- C30, C31, C32, C33, C34, C35, C36: footprint (none) -> Capacitor_SMD:C_0603_1608Metric_Pad1.05x0.95mm_HandSolder
- R7, R8: footprint (none) -> Resistor_SMD:R_0805_2012Metric_Pad1.15x1.40mm_HandSolder
Changed lines of the file:
@@
 F 0 "R7" H 3750 3750 50  0000 L CNN
 F 1 "49.9" H 3800 3600 50  0000 L CNN
-F 2 "" V 3830 3650 50  0001 C CNN
+F 2 "Resistor_SMD:R_0805_2012Metric_Pad1.15x1.40mm_HandSolder" V 3830 3650 50  0001 C CNN
 F 3 "~" H 3900 3650 50  0001 C CNN
 	1    3900 3650
@@
 F 0 "C31" H 4250 3550 50  0000 R CNN
 F 1 "0.1u" H 4200 3750 50  0000 R CNN
-F 2 "" H 4188 3500 50  0001 C CNN
+F 2 "Capacitor_SMD:C_0603_1608Metric_Pad1.05x0.95mm_HandSolder" H 4188 3500 50  0001 C CNN
 F 3 "~" H 4150 3650 50  0001 C CNN
 	1    4150 3650
@@
 F 0 "R8" H 4250 3750 50  0000 L CNN
 F 1 "24.9" H 4300 3600 50  0000 L CNN
-F 2 "" V 4330 3650 50  0001 C CNN
+F 2 "Resistor_SMD:R_0805_2012Metric_Pad1.15x1.40mm_HandSolder" V 4330 3650 50  0001 C CNN
 F 3 "~" H 4400 3650 50  0001 C CNN
 	1    4400 3650
@@
 F 0 "C34" H 5000 4450 50  0000 R CNN
 F 1 "0.1u" H 4950 4650 50  0000 R CNN
-F 2 "" H 4938 4400 50  0001 C CNN
+F 2 "Capacitor_SMD:C_0603_1608Metric_Pad1.05x0.95mm_HandSolder" H 4938 4400 50  0001 C CNN
 F 3 "~" H 4900 4550 50  0001 C CNN
 	1    4900 4550
@@
 F 0 "C35" H 5400 4450 50  0000 R CNN
 F 1 "10u" H 5350 4650 50  0000 R CNN
-F 2 "" H 5338 4400 50  0001 C CNN
+F 2 "Capacitor_SMD:C_0603_1608Metric_Pad1.05x0.95mm_HandSolder" H 5338 4400 50  0001 C CNN
 F 3 "~" H 5300 4550 50  0001 C CNN
 	1    5300 4550
@@
 F 0 "C36" H 6050 3650 50  0000 R CNN
 F 1 "10n" H 6000 3850 50  0000 R CNN
-F 2 "" H 5988 3600 50  0001 C CNN
+F 2 "Capacitor_SMD:C_0603_1608Metric_Pad1.05x0.95mm_HandSolder" H 5988 3600 50  0001 C CNN
 F 3 "~" H 5950 3750 50  0001 C CNN
 	1    5950 3750
@@
 F 0 "C30" H 4150 2600 50  0000 R CNN
 F 1 "0.1u" H 4100 2800 50  0000 R CNN
-F 2 "" H 4088 2550 50  0001 C CNN
+F 2 "Capacitor_SMD:C_0603_1608Metric_Pad1.05x0.95mm_HandSolder" H 4088 2550 50  0001 C CNN
 F 3 "~" H 4050 2700 50  0001 C CNN
 	1    4050 2700
@@
 F 0 "C32" H 4400 2600 50  0000 R CNN
 F 1 "10u" H 4350 2800 50  0000 R CNN
-F 2 "" H 4338 2550 50  0001 C CNN
+F 2 "Capacitor_SMD:C_0603_1608Metric_Pad1.05x0.95mm_HandSolder" H 4338 2550 50  0001 C CNN
 F 3 "~" H 4300 2700 50  0001 C CNN
 	1    4300 2700
@@
 F 0 "C33" H 4700 3550 50  0000 R CNN
 F 1 "10n" H 4650 3750 50  0000 R CNN
-F 2 "" H 4638 3500 50  0001 C CNN
+F 2 "Capacitor_SMD:C_0603_1608Metric_Pad1.05x0.95mm_HandSolder" H 4638 3500 50  0001 C CNN
 F 3 "~" H 4600 3650 50  0001 C CNN
 	1    4600 3650
