File: 8330EVA-kicad/USB2SPI.sch (KiCad schematic (older format))
At the start: 28 parts, among them U1 AMS1117-3.3, U2 FT232H, Y1 12Mhz

Commit message: 为变压器制作封装
Parts:
- C14, C15, C16: footprint (none) -> Capacitor_SMD:C_0603_1608Metric_Pad1.05x0.95mm_HandSolder
Changed lines of the file:
@@
 F 0 "C14" H 1215 5546 50  0000 L CNN
 F 1 "4.7u" H 1215 5455 50  0000 L CNN
-F 2 "" H 1138 5350 50  0001 C CNN
+F 2 "Capacitor_SMD:C_0603_1608Metric_Pad1.05x0.95mm_HandSolder" H 1138 5350 50  0001 C CNN
 F 3 "~" H 1100 5500 50  0001 C CNN
 	1    1100 5500
@@
 F 0 "C15" H 1765 5546 50  0000 L CNN
 F 1 "100n" H 1765 5455 50  0000 L CNN
-F 2 "" H 1688 5350 50  0001 C CNN
+F 2 "Capacitor_SMD:C_0603_1608Metric_Pad1.05x0.95mm_HandSolder" H 1688 5350 50  0001 C CNN
 F 3 "~" H 1650 5500 50  0001 C CNN
 	1    1650 5500
@@
 F 0 "C16" H 2615 5546 50  0000 L CNN
 F 1 "100n" H 2550 5400 50  0000 L CNN
-F 2 "" H 2538 5350 50  0001 C CNN
+F 2 "Capacitor_SMD:C_0603_1608Metric_Pad1.05x0.95mm_HandSolder" H 2538 5350 50  0001 C CNN
 F 3 "~" H 2500 5500 50  0001 C CNN
 	1    2500 5500
