File: 8330EVA-kicad/8330_EVA.sch (KiCad schematic (older format))
At the start: 5 parts, among them J1 USB_B_Micro, J2 Conn_Coaxial, J3 Conn_01x03_Male, J4 Conn_Coaxial, J5 Conn_Coaxial

Commit message: 更新3d模型，替换SMA接头的封装
Parts:
- J1: footprint Connector_USB:USB_Micro-B_Wuerth_614105150721_Vertical -> Connector_USB:USB_Micro-B_Molex_47346-0001
- J2: footprint Connector_Coaxial:SMA_Amphenol_132289_EdgeMount -> Connector_Coaxial:SMA_Amphenol_132134-14_Vertical
- J4, J5: footprint Connector_Coaxial:SMA_Amphenol_132289_EdgeMount -> Connector_Coaxial:SMA_Amphenol_132134-11_Vertical
Changed lines of the file:
@@
 F 0 "J2" H 3550 4050 50  0000 L CNN
 F 1 "Conn_Coaxial" H 3500 3734 50  0000 L CNN
-F 2 "Connector_Coaxial:SMA_Amphenol_132289_EdgeMount" H 3400 3850 50  0001 C CNN
+F 2 "Connector_Coaxial:SMA_Amphenol_132134-14_Vertical" H 3400 3850 50  0001 C CNN
 F 3 " ~" H 3400 3850 50  0001 C CNN
 	1    3400 3850
@@
 F 0 "J4" H 7550 3582 50  0000 L CNN
 F 1 "Conn_Coaxial" H 7550 3673 50  0000 L CNN
-F 2 "Connector_Coaxial:SMA_Amphenol_132289_EdgeMount" H 7450 3700 50  0001 C CNN
+F 2 "Connector_Coaxial:SMA_Amphenol_132134-11_Vertical" H 7450 3700 50  0001 C CNN
 F 3 " ~" H 7450 3700 50  0001 C CNN
 	1    7450 3700
@@
 F 0 "J5" H 7550 3875 50  0000 L CNN
 F 1 "Conn_Coaxial" H 7550 3784 50  0000 L CNN
-F 2 "Connector_Coaxial:SMA_Amphenol_132289_EdgeMount" H 7450 3900 50  0001 C CNN
+F 2 "Connector_Coaxial:SMA_Amphenol_132134-11_Vertical" H 7450 3900 50  0001 C CNN
 F 3 " ~" H 7450 3900 50  0001 C CNN
 	1    7450 3900
@@
 F 0 "J1" H 1620 5097 50  0000 R CNN
 F 1 "USB_B_Micro" H 1620 5188 50  0000 R CNN
-F 2 "Connector_USB:USB_Micro-B_Wuerth_614105150721_Vertical" H 2000 5150 50  0001 C CNN
+F 2 "Connector_USB:USB_Micro-B_Molex_47346-0001" H 2000 5150 50  0001 C CNN
 F 3 "~" H 2000 5150 50  0001 C CNN
 	1    1850 5200

Commit message: Finished PCB layout, connect Earth to Ground
Parts:
- J1: footprint Connector_USB:USB_Micro-B_Molex_47346-0001 -> Connector_USB:USB_Micro-B_Wuerth_614105150721_Vertical
- J2: footprint Connector_Coaxial:SMA_Amphenol_132134-14_Vertical -> Connector_Coaxial:SMA_Amphenol_132289_EdgeMount
- J4, J5: footprint Connector_Coaxial:SMA_Amphenol_132134-11_Vertical -> Connector_Coaxial:SMA_Amphenol_132289_EdgeMount
Connections:
- net USB2SPI/Ground is gone; now on net Earth: J1.5 (GND), J1.6 (Shield)
Changed lines of the file:
@@
 EESchema Schematic File Version 4
 LIBS:8330_EVA-cache
-EELAYER 29 0
+EELAYER 26 0
 EELAYER END
 $Descr A4 11693 8268
@@
 F6 "VCC_+5V" I L 5850 3500 50
 F7 "VEE_-5V" I L 5850 3600 50
-F8 "GROUND" I L 5850 4200 50
+F8 "Earth" I L 5850 4200 50
 F9 "SignalIN" I L 5850 3850 50
 $EndSheet
@@
 F 0 "J2" H 3550 4050 50  0000 L CNN
 F 1 "Conn_Coaxial" H 3500 3734 50  0000 L CNN
-F 2 "Connector_Coaxial:SMA_Amphenol_132134-14_Vertical" H 3400 3850 50  0001 C CNN
+F 2 "Connector_Coaxial:SMA_Amphenol_132289_EdgeMount" H 3400 3850 50  0001 C CNN
 F 3 " ~" H 3400 3850 50  0001 C CNN
 	1    3400 3850
@@
 F 0 "J4" H 7550 3582 50  0000 L CNN
 F 1 "Conn_Coaxial" H 7550 3673 50  0000 L CNN
-F 2 "Connector_Coaxial:SMA_Amphenol_132134-11_Vertical" H 7450 3700 50  0001 C CNN
+F 2 "Connector_Coaxial:SMA_Amphenol_132289_EdgeMount" H 7450 3700 50  0001 C CNN
 F 3 " ~" H 7450 3700 50  0001 C CNN
 	1    7450 3700
@@
 F 0 "J5" H 7550 3875 50  0000 L CNN
 F 1 "Conn_Coaxial" H 7550 3784 50  0000 L CNN
-F 2 "Connector_Coaxial:SMA_Amphenol_132134-11_Vertical" H 7450 3900 50  0001 C CNN
+F 2 "Connector_Coaxial:SMA_Amphenol_132289_EdgeMount" H 7450 3900 50  0001 C CNN
 F 3 " ~" H 7450 3900 50  0001 C CNN
 	1    7450 3900
@@
 	2500 4050 2500 5750
 Wire Wire Line
-	2500 5750 4150 5750
+	2500 5750 2650 5750
 Connection ~ 4150 5750
 Connection ~ 5350 5750
@@
 F 0 "J1" H 1620 5097 50  0000 R CNN
 F 1 "USB_B_Micro" H 1620 5188 50  0000 R CNN
-F 2 "Connector_USB:USB_Micro-B_Molex_47346-0001" H 2000 5150 50  0001 C CNN
+F 2 "Connector_USB:USB_Micro-B_Wuerth_614105150721_Vertical" H 2000 5150 50  0001 C CNN
 F 3 "~" H 2000 5150 50  0001 C CNN
 	1    1850 5200
@@
 	3050 5400 2150 5400
 Wire Wire Line
-	2250 5550 3050 5550
+	2250 5550 2650 5550
 Wire Wire Line
 	1750 4800 1750 4650
@@
 Connection ~ 1850 4650
 NoConn ~ 2150 5000
+Wire Wire Line
+	2650 5550 2650 5750
+Connection ~ 2650 5550
+Wire Wire Line
+	2650 5550 3050 5550
+Connection ~ 2650 5750
+Wire Wire Line
+	2650 5750 4150 5750
 $EndSCHEMATC
