File: 8330EVA-kicad/8330_EVA.sch (KiCad schematic (older format))
At the start: 5 parts, among them J1 USB_B_Micro, J2 Conn_Coaxial, J3 Conn_01x03_Male, J4 Conn_Coaxial, J5 Conn_Coaxial

Commit message: 简单修改
1. 修改了差分输出处的布线，提高对称性
2. 修改了USB接口的封装。现在使用完全表面贴装的Mini USB接口
3. 在电路板上添加了要求的信息
4. 生成了BOM表和Gerber文件
Parts:
- J1: footprint Connector_USB:USB_Micro-B_Wuerth_614105150721_Vertical -> Connector_USB:USB_Mini-B_Lumberg_2486_01_Horizontal
Changed lines of the file:
@@
 EESchema Schematic File Version 4
 LIBS:8330_EVA-cache
-EELAYER 26 0
+EELAYER 29 0
 EELAYER END
 $Descr A4 11693 8268
@@
 F 0 "J1" H 1620 5097 50  0000 R CNN
 F 1 "USB_B_Micro" H 1620 5188 50  0000 R CNN
-F 2 "Connector_USB:USB_Micro-B_Wuerth_614105150721_Vertical" H 2000 5150 50  0001 C CNN
+F 2 "Connector_USB:USB_Mini-B_Lumberg_2486_01_Horizontal" H 2000 5150 50  0001 C CNN
 F 3 "~" H 2000 5150 50  0001 C CNN
 	1    1850 5200
